Commit message: complete the surface fitting moudle

File: src/uam_control_interface/urdf/skyvortex.urdf (robot description, URDF)
Before this commit: robot skyvortex, 8 links, 7 joints
Links:
- removed link operator_1_Link_collision
- removed link robot_base
- removed link rotor_0_collision_respondable
- removed link rotor_1_collision_respondable
- removed link rotor_2_collision_respondable
- removed link rotor_3_collision_respondable
- removed link rotor_4_collision_respondable
- removed link rotor_5_collision_respondable
- added link base_link, mass 2.10772457717204; collision mesh filename=package://uam_control_interface/urdf/mesh/base_link.STL; visual mesh filename=package://uam_control_interface/urdf/mesh/base_link.STL
- added link camera_Link, mass 1.26688452104529; collision mesh filename=package://uam_control_interface/urdf/mesh/camera_Link.STL; visual mesh filename=package://uam_control_interface/urdf/mesh/camera_Link.STL
- added link depth_optical_frame
- added link end_Link, mass 3.14159265358975E-06; collision mesh filename=package://uam_control_interface/urdf/mesh/end_Link.STL; visual mesh filename=package://uam_control_interface/urdf/mesh/end_Link.STL
- added link operator_Link, mass 1.53399501100992; collision mesh filename=package://uam_control_interface/urdf/mesh/operator_Link.STL; visual mesh filename=package://uam_control_interface/urdf/mesh/operator_Link.STL
- added link rotor1_Link, mass 0.0159144165937803; collision mesh filename=package://uam_control_interface/urdf/mesh/rotor1_Link.STL; visual mesh filename=package://uam_control_interface/urdf/mesh/rotor1_Link.STL
- added link rotor2_Link, mass 0.0159143233965928; collision mesh filename=package://uam_control_interface/urdf/mesh/rotor2_Link.STL; visual mesh filename=package://uam_control_interface/urdf/mesh/rotor2_Link.STL
- added link rotor3_Link, mass 0.0159143198305425; collision mesh filename=package://uam_control_interface/urdf/mesh/rotor3_Link.STL; visual mesh filename=package://uam_control_interface/urdf/mesh/rotor3_Link.STL
- added link rotor4_Link, mass 0.0159142814024756; collision mesh filename=package://uam_control_interface/urdf/mesh/rotor4_Link.STL; visual mesh filename=package://uam_control_interface/urdf/mesh/rotor4_Link.STL
- added link rotor5_Link, mass 0.0159143909446094; collision mesh filename=package://uam_control_interface/urdf/mesh/rotor5_Link.STL; visual mesh filename=package://uam_control_interface/urdf/mesh/rotor5_Link.STL
- added link rotor6_Link, mass 0.0159142602415204; collision mesh filename=package://uam_control_interface/urdf/mesh/rotor6_Link.STL; visual mesh filename=package://uam_control_interface/urdf/mesh/rotor6_Link.STL
Joints:
- added joint camera_joint: type fixed, parent operator_Link, child camera_Link, origin xyz=-0.1084 0.001842 0.21154 rpy=0 -0.5236 -0.016991, axis 0 0 0
- added joint depth_optical_frame: type fixed, parent camera_Link, child depth_optical_frame, origin xyz=0 0 0 rpy=-1.570796 0 -1.570796, axis 0 0 0
- added joint end_Link: type fixed, parent operator_Link, child end_Link, origin xyz=0.832190790551214 -0.0141410330369185 0.480534938269667 rpy=0 1.04719755119663 -0.0169909387168526, axis 0 0 0
- joint operator_1_joint: axis 0 0 1 -> -0.016990083887519 -0.999855658107456 0; child operator_1_Link_collision -> operator_Link; limit (none) -> lower=0 upper=0 effort=0 velocity=0; origin xyz=1.689620 2.000172 1.003455 rpy=-1.570796 3.158584 3.124602 -> xyz=0.000870575084399361 0.000171621257114271 0.0284550617303106 rpy=0 0 0; parent robot_base -> base_link; type continuous -> revolute
- joint rotor_0_joint: axis 0 0 1 -> -0.25 0.43301 0.86603; child rotor_0_collision_respondable -> rotor1_Link; limit lower=-100000.0 upper=74532.925199444 effort=10.0 velocity=1e6 -> lower=0 upper=0 effort=0 velocity=0; origin xyz=2.130819 2.277801 1.008856 rpy=2.677950 3.394273 -3.081642 -> xyz=0.44207 0.2778 0.033856 rpy=0 0 0; parent robot_base -> base_link; type fixed -> revolute
- joint rotor_1_joint: axis 0 0 1 -> 0.5 0 0.86603; child rotor_1_collision_respondable -> rotor2_Link; limit lower=-100000.0 upper=74532.925199444 effort=10.0 velocity=1e6 -> lower=0 upper=0 effort=0 velocity=0; origin xyz=1.708297 2.521750 1.008857 rpy=-3.141592 2.617997 3.141592 -> xyz=0.019547 0.52175 0.033856 rpy=0 0 0; parent robot_base -> base_link; type fixed -> revolute
- joint rotor_2_joint: axis 0 0 1 -> -0.25 -0.43301 0.86603; child rotor_2_collision_respondable -> rotor3_Link; limit lower=-100000.0 upper=74532.925199444 effort=10.0 velocity=1e6 -> lower=0 upper=0 effort=0 velocity=0; origin xyz=1.227130 2.243950 1.008856 rpy=-2.677949 3.394273 3.081642 -> xyz=-0.46162 0.24395 0.033856 rpy=0 0 0; parent robot_base -> base_link; type fixed -> revolute
- joint rotor_3_joint: axis 0 0 1 -> -0.25 0.43301 0.86603; child rotor_3_collision_respondable -> rotor4_Link; limit lower=-100000.0 upper=74532.925199444 effort=10.0 velocity=1e6 -> lower=0 upper=0 effort=0 velocity=0; origin xyz=1.227129 1.756050 1.008856 rpy=2.677950 3.394273 -3.081642 -> xyz=-0.46162 -0.24395 0.033856 rpy=0 0 0; parent robot_base -> base_link; type fixed -> revolute
- joint rotor_4_joint: axis 0 0 1 -> 0.5 0 0.86603; child rotor_4_collision_respondable -> rotor5_Link; limit lower=-100000.0 upper=74532.925199444 effort=10.0 velocity=1e6 -> lower=0 upper=0 effort=0 velocity=0; origin xyz=1.708296 1.478250 1.008856 rpy=-3.141592 2.617997 3.141592 -> xyz=0.019547 -0.52175 0.033856 rpy=0 0 0; parent robot_base -> base_link; type fixed -> revolute
- joint rotor_5_joint: axis 0 0 1 -> -0.250000000000029 -0.433012701892223 0.866025403784428; child rotor_5_collision_respondable -> rotor6_Link; limit lower=-100000.0 upper=74532.925199444 effort=10.0 velocity=1e6 -> lower=0 upper=0 effort=0 velocity=0; origin xyz=2.130819 1.722200 1.008856 rpy=-2.677949 3.394273 3.081642 -> xyz=0.442073608231067 -0.277801787065658 0.0338557055276746 rpy=0 0 0; parent robot_base -> base_link; type fixed -> revolute

Commit message: update the urdf files, which has included the end_effector

File: src/uam_control_interface/urdf/skyvortex.urdf (robot description, URDF)
Before this commit: robot uma3_.SLDASM2, 11 links, 10 joints
Links:
- added link connect_Link, mass 0.049595; collision mesh filename=package://uam_control_interface/urdf/mesh/connect_Link.STL; visual mesh filename=package://uam_control_interface/urdf/mesh/connect_Link.STL
- added link end_effector_base_Link, mass 0.015757; collision mesh filename=package://uam_control_interface/urdf/mesh/end_effector_base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; visual mesh filename=package://uam_control_interface/urdf/mesh/end_effector_base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
- added link move_base_Link, mass 0.17494; collision mesh filename=package://uam_control_interface/urdf/mesh/move_base_Link.STL; visual mesh filename=package://uam_control_interface/urdf/mesh/move_base_Link.STL
- added link wheel1_Link, mass 0.041284; collision mesh filename=package://uam_control_interface/urdf/mesh/wheel1_Link.STL; visual mesh filename=package://uam_control_interface/urdf/mesh/wheel1_Link.STL
- added link wheel2_Link, mass 0.040979; collision mesh filename=package://uam_control_interface/urdf/mesh/wheel2_Link.STL; visual mesh filename=package://uam_control_interface/urdf/mesh/wheel2_Link.STL
- added link wheel3_Link, mass 0.040979; collision mesh filename=package://uam_control_interface/urdf/mesh/wheel3_Link.STL; visual mesh filename=package://uam_control_interface/urdf/mesh/wheel3_Link.STL
Joints:
- added joint connect_joint: type prismatic, parent end_effector_base_Link, child connect_Link, origin xyz=0 0 -0.29735 rpy=0 0 0, axis 0 0 1, limit lower=0 upper=0 effort=0 velocity=0
- added joint end_effector_joint: type fixed, parent operator_Link, child end_effector_base_Link, origin xyz=0.257683193140019 -0.00437869126722494 0.148794938269686 rpy=2.09439510239316 0 -1.58778722885262, axis 0 0 0
- added joint move_base_joint: type fixed, parent connect_Link, child move_base_Link, origin xyz=0 0 -0.4115 rpy=0 0 0, axis 0 0 0
- added joint wheel1_joint: type continuous, parent move_base_Link, child wheel1_Link, origin xyz=0 0.085482 0.0115 rpy=0 0 0, axis 0 1 0
- added joint wheel2_joint: type continuous, parent move_base_Link, child wheel2_Link, origin xyz=0.07403 -0.042741 0.0115 rpy=0 0 -2.0944, axis 0 1 0
- added joint wheel3_joint: type continuous, parent move_base_Link, child wheel3_Link, origin xyz=-0.07403 -0.042741 0.0115 rpy=0 0 2.0944, axis 0 1 0
